Commit message: fixed typo, changed update rates for sensors

File: rosws/src/simple_cube/urdf/simple_cube_hector.urdf (robot description, URDF)
Before this commit: robot simple_cube_hector, 1 links, 0 joints
Links:
- link base_link: mass 0.001 -> 0.1

Commit message: changed update rate for sensors in simple_cube_hector

File: rosws/src/simple_cube/urdf/simple_cube_hector.urdf (robot description, URDF)
Before this commit: robot simple_cube_hector, 1 links, 0 joints
Links:
- link base_link: mass 0.1 -> 0.01

Commit message: added and rotated imu_link in simple_cuble_hector.urdf

File: rosws/src/simple_cube/urdf/simple_cube_hector.urdf (robot description, URDF)
Before this commit: robot simple_cube_hector, 1 links, 0 joints
Links:
- added link imu_link
Joints:
- added joint imu_joint: type fixed, parent base_link, child imu_link, origin xyz=0 0 0 rpy=3.141592653 0 1.570796326
