Commit message: rotated imu_link

File: rosws/src/turtlebot3_description/urdf/turtlebot3_burger.urdf.xacro (robot description, xacro)
@@ -110,5 +110,5 @@
     <parent link="base_link"/>
     <child link="imu_link"/>
-    <origin xyz="-0.032 0 0.068" rpy="0 0 0"/>
+    <origin xyz="-0.032 0 0.068" rpy=rpy="3.141592653 0 1.570796326"/>
   </joint>
   <link name="imu_link"/>

Commit message: fixed a bug in the urdf xacro for turtlebot; implemented position estimation + plot inside GUI

File: rosws/src/turtlebot3_description/urdf/turtlebot3_burger.urdf.xacro (robot description, xacro)
@@ -110,5 +110,5 @@
     <parent link="base_link"/>
     <child link="imu_link"/>
-    <origin xyz="-0.032 0 0.068" rpy=rpy="3.141592653 0 1.570796326"/>
+    <origin xyz="-0.032 0 0.068" rpy="3.141592653 0 1.570796326"/>
   </joint>
   <link name="imu_link"/>

Commit message: fixed a bug in 2d plot where the mag-z axis was confused with mag-x

File: rosws/src/turtlebot3_description/urdf/turtlebot3_burger.urdf.xacro (robot description, xacro)
@@ -112,5 +112,7 @@
     <origin xyz="-0.032 0 0.068" rpy="3.141592653 0 1.570796326"/>
   </joint>
-  <link name="imu_link"/>
+  <link name="imu_link">
+    <origin xyz="-0.032 0 0.068" rpy="0 0 0"/>
+  </link>
   <joint name="scan_joint" type="fixed">
     <parent link="base_link"/>

Commit message: changed imu_link rotation to 0

File: rosws/src/turtlebot3_description/urdf/turtlebot3_burger.urdf.xacro (robot description, xacro)
@@ -110,8 +110,8 @@
     <parent link="base_link"/>
     <child link="imu_link"/>
-    <origin xyz="-0.032 0 0.068" rpy="3.141592653 0 1.570796326"/>
+    <origin xyz="-0.032 0 0.068" rpy="0 0 0"/>
   </joint>
   <link name="imu_link">
-    <origin xyz="-0.032 0 0.068" rpy="0 0 0"/>
+    <origin xyz="0 0 0" rpy="0 0 0"/>
   </link>
   <joint name="scan_joint" type="fixed">
